Commit message: latest

File: src/oribot_description/src/description/oribot_description.urdf (robot description, URDF)
Before this commit: robot oribot, 5 links, 4 joints
Links:
- removed link camera_depth_frame
- removed link camera_link
- removed link lidar_link
- added link imu_link; visual box size=${imu_length} ${imu_width} ${imu_height}
- added link laser, mass 0.125; collision cylinder length=0.055 radius=0.0508; visual cylinder length=0.055 radius=0.0508
Joints:
- removed joint camera_depth_joint
- removed joint camera_joint
- added joint imu_joint: type fixed, parent base_link, child imu_link, origin xyz=${imu_xoff} 0 ${imu_zoff} rpy=0 0 0
- joint lidar_joint: child lidar_link -> laser; origin xyz=0 0 0.12 rpy=0 0 0 -> xyz=${lidar_xoff} 0 ${lidar_zoff} rpy=0 0 ${pi}

Commit message: latest

File: src/oribot_description/src/description/oribot_description.urdf (robot description, URDF)
Before this commit: robot oribot, 4 links, 3 joints
Links:
- added link camera; visual box size=0.02 0.02 0.02
Joints:
- added joint camera_joint: type fixed, parent base_link, child camera, origin xyz=${base_length/2.0 + 0.01} 0 ${base_height/2.0 - 0.01} rpy=0 0 0
